Commit message: packages cleanup

File: src/velmobil_description/urdf/simple_velmobil.urdf.xacro (robot description, xacro)
@@ -1,7 +1,6 @@
 <?xml version="1.0"?>
 <robot name="simple_velmobil" xmlns:xacro="http://www.ros.org/wiki/xacro" xmlns:gz="http://gazebosim.org/schema">
-  <material name="orange"><color rgba="0.8 0.4 0.0 1.0"/></material>
-  <material name="black"><color rgba="0 0 0 1.0"/></material>
-  <material name="white"><color rgba="1 1 1 1.0"/></material>
+  <xacro:include filename="$(find velmobil_description)/urdf/properties.urdf.xacro" />
+  <xacro:include filename="$(find velmobil_description)/urdf/macros.urdf.xacro" />
   <link name="base_link">
     <collision>
@@ -20,40 +19,8 @@
     </inertial>
   </link>
-  <xacro:macro name="wheel" params="prefix x y">
-    <joint name="${prefix}_wheel_joint" type="continuous">
-      <origin xyz="${x} ${y} 0.3" rpy="-${pi/2} 0 0"/>
-      <parent link="base_link"/>
-      <child link="${prefix}_wheel"/>
-      <axis xyz="0 0 1"/>
-      <dynamics damping="0.2"/>
-    </joint>
-    <link name="${prefix}_wheel">
-      <collision><geometry><sphere radius="0.3"/></geometry></collision>
-      <visual><geometry><sphere radius="0.3"/></geometry><material name="black"/></visual>
-      <inertial>
-        <mass value="2"/>
-        <inertia ixx="0.145" ixy="0.0" ixz="0.0" iyy="0.145" iyz="0.0" izz="0.125"/>
-      </inertial>
-    </link>
-  </xacro:macro>
   <xacro:wheel prefix="front_left" x="0.6" y="0.5"/>
   <xacro:wheel prefix="front_right" x="0.6" y="-0.5"/>
   <xacro:wheel prefix="rear_left" x="-0.6" y="0.5"/>
   <xacro:wheel prefix="rear_right" x="-0.6" y="-0.5"/>
-  <xacro:macro name="wheel_friction" params="prefix dir">
-    <gazebo reference="${prefix}_wheel">
-      <collision>
-        <surface>
-          <friction>
-            <ode>
-              <mu1>1.0</mu1><mu2>1.0</mu2>
-              <kp>1000000.0</kp><kd>10.0</kd><minDepth>0.001</minDepth>
-              <fdir1 gz:expressed_in="base_link">1 ${dir} 0</fdir1>
-            </ode>
-          </friction>
-        </surface>
-      </collision>
-    </gazebo>
-  </xacro:macro>
   <xacro:wheel_friction prefix="front_left" dir="-1"/>
   <xacro:wheel_friction prefix="front_right" dir="1"/>
@@ -62,10 +29,4 @@
   <ros2_control name="GazeboSimSystem" type="system">
     <hardware><plugin>gz_ros2_control/GazeboSimSystem</plugin></hardware>
-    <xacro:macro name="joint_interface" params="name">
-      <joint name="${name}">
-        <command_interface name="velocity"><param name="min">-1</param><param name="max">1</param></command_interface>
-        <state_interface name="position"/><state_interface name="velocity"/>
-      </joint>
-    </xacro:macro>
     <xacro:joint_interface name="front_left_wheel_joint"/>
     <xacro:joint_interface name="front_right_wheel_joint"/>
@@ -75,5 +36,5 @@
   <gazebo>
     <plugin filename="gz_ros2_control-system" name="gz_ros2_control::GazeboSimROS2ControlPlugin">
-      <parameters>$(find velmobil)/config/simple_velmobil.yaml</parameters>
+      <parameters>$(find velmobil_description)/control/simple_velmobil.yaml</parameters>
       <ros>
         <remapping>/mecanum_drive_controller/reference:=/cmd_vel</remapping>
