Commit message: velmobil doesnt move Y yet

File: src/velmobil_description/urdf/macros.urdf.xacro (robot description, xacro)
@@ -2,19 +2,28 @@
 <robot name="simple_velmobil" xmlns:xacro="http://www.ros.org/wiki/xacro" xmlns:gz="http://gazebosim.org/schema">
     <xacro:macro name="wheel" params="prefix x y">
-        <joint name="${prefix}_wheel_joint" type="continuous">
-            <origin xyz="${x} ${y} 0.3" rpy="-${pi/2} 0 0"/>
-            <parent link="base_link"/>
-            <child link="${prefix}_wheel"/>
-            <axis xyz="0 0 1"/>
-            <dynamics damping="0.2"/>
-        </joint>
         <link name="${prefix}_wheel">
-            <collision><geometry><sphere radius="0.3"/></geometry></collision>
-            <visual><geometry><sphere radius="0.3"/></geometry><material name="black"/></visual>
+            <collision>
+                <origin xyz="0 0 0" rpy="${-pi/2} 0 0"/>
+                <geometry><cylinder length="0.1" radius="${wheel_radius}"/></geometry>
+            </collision>
+            <visual>
+                <origin xyz="0 0 0" rpy="${-pi/2} 0 0"/>
+                <geometry>
+                    <cylinder length="0.1" radius="${wheel_radius}"/>
+                </geometry>
+                <material name="black"/>
+            </visual>
             <inertial>
-                <mass value="2"/>
+                <mass value="1.0"/>
                 <inertia ixx="0.145" ixy="0.0" ixz="0.0" iyy="0.145" iyz="0.0" izz="0.125"/>
             </inertial>
         </link>
+        <joint name="${prefix}_wheel_joint" type="continuous">
+            <origin xyz="${x} ${y} ${-wheel_base_offset}" rpy="0 0 0"/>
+            <parent link="base_link"/>
+            <child link="${prefix}_wheel"/>
+            <axis xyz="0 1 0"/>
+            <dynamics damping="0.2"/>
+        </joint>
     </xacro:macro>
     <xacro:macro name="wheel_friction" params="prefix dir">
@@ -22,13 +31,23 @@
             <collision>
                 <surface>
-                <friction>
-                    <ode>
-                        <mu1>1.0</mu1><mu2>1.0</mu2>
-                        <kp>1000000.0</kp><kd>10.0</kd><minDepth>0.001</minDepth>
-                        <fdir1 gz:expressed_in="base_link">1 ${dir} 0</fdir1>
-                    </ode>
-                </friction>
+                    <friction>
+                        <ode>
+                            <mu>1.0</mu>
+                            <mu2>0.01</mu2>
+                            <fdir1>1 ${dir} 0</fdir1>
+                            <slip1>0.0</slip1>
+                            <slip2>0.5</slip2>
+                        </ode>
+                    </friction>
+                    <contact>
+                        <ode>
+                            <kp>1000000.0</kp>
+                            <kd>1.0</kd>
+                            <min_depth>0.001</min_depth>
+                        </ode>
+                    </contact>
                 </surface>
             </collision>
+            <selfCollide>false</selfCollide>
         </gazebo>
     </xacro:macro>
@@ -36,6 +55,6 @@
         <joint name="${name}">
             <command_interface name="velocity">
-                <param name="min">-1</param>
-                <param name="max">1</param>
+                <param name="min">-10000</param>
+                <param name="max">10000</param>
             </command_interface>
             <state_interface name="position"/>

File: src/velmobil_description/urdf/properties.urdf.xacro (robot description, xacro)
@@ -4,3 +4,14 @@
     <material name="black"><color rgba="0 0 0 1.0"/></material>
     <material name="white"><color rgba="1 1 1 1.0"/></material>
+    <xacro:property name="wheel_radius" value="0.1016"/>
+    <xacro:property name="lidar_l_centre_offset" value="0 0.3 0.176"/>
+    <xacro:property name="lidar_l_orientation" value="0 0 0"/>
+    <xacro:property name="lidar_r_centre_offset" value="0 -0.3 0.176"/>
+    <xacro:property name="lidar_r_orientation" value="0 0 -3.141592"/>
+    <xacro:property name="imu_centre_ofset" value="0 0 0"/>
+    <xacro:property name="wheel_y_offset" value="0.38"/>
+    <xacro:property name="wheel_centre_x_offset" value="0.36"/>
+    <xacro:property name="wheel_r_base_x_offset" value="${-wheel_centre_x_offset + 0.081}"/>
+    <xacro:property name="wheel_f_front_x_offset" value="${0.445 - 0.081 - wheel_centre_x_offset}"/>
+    <xacro:property name="wheel_base_offset" value="0.05"/>
 </robot>

File: src/velmobil_description/urdf/simple_velmobil.urdf.xacro (robot description, xacro)
@@ -3,28 +3,34 @@
   <xacro:include filename="$(find velmobil_description)/urdf/properties.urdf.xacro" />
   <xacro:include filename="$(find velmobil_description)/urdf/macros.urdf.xacro" />
+  <link name="base_footprint" />
   <link name="base_link">
     <collision>
       <origin xyz="0 0 0.5" rpy="0 0 0"/>
-      <geometry><box size="2 1 0.5"/></geometry>
+      <geometry><box size="0.1 0.1 0.1"/></geometry>  <!-- mock colision -->
     </collision>
     <visual>
-      <origin xyz="0 0 0.5" rpy="0 0 0"/>
-      <geometry><box size="2 1 0.5"/></geometry>
-      <material name="orange"/>
+      <geometry>
+        <mesh filename="file://$(find velmobil_description)/models/base.dae" />
+      </geometry>
     </visual>
     <inertial>
       <origin xyz="0 0 0.5" rpy="0 0 0"/>
-      <mass value="1.5"/>
+      <mass value="0.5"/>
       <inertia ixx="0.13" ixy="0.0" ixz="0.0" iyy="0.42" iyz="0.0" izz="0.48"/>
     </inertial>
   </link>
-  <xacro:wheel prefix="front_left" x="0.6" y="0.5"/>
-  <xacro:wheel prefix="front_right" x="0.6" y="-0.5"/>
-  <xacro:wheel prefix="rear_left" x="-0.6" y="0.5"/>
-  <xacro:wheel prefix="rear_right" x="-0.6" y="-0.5"/>
-  <xacro:wheel_friction prefix="front_left" dir="-1"/>
-  <xacro:wheel_friction prefix="front_right" dir="1"/>
-  <xacro:wheel_friction prefix="rear_left" dir="1"/>
-  <xacro:wheel_friction prefix="rear_right" dir="-1"/>
+  <joint name="footprint_joint" type="fixed">
+      <origin xyz="0 0 ${wheel_radius + wheel_base_offset}" rpy="0 0 0"/>
+      <parent link="base_footprint"/>
+      <child link="base_link"/>
+  </joint>
+  <xacro:wheel prefix="front_left" x="0.5" y="${wheel_y_offset}"/>
+  <xacro:wheel prefix="front_right" x="0.5" y="${-wheel_y_offset}"/>
+  <xacro:wheel prefix="rear_left" x="-0.5" y="${wheel_y_offset}"/>
+  <xacro:wheel prefix="rear_right" x="-0.5" y="${-wheel_y_offset}"/>
+  <xacro:wheel_friction prefix="front_left" dir="1"/>
+  <xacro:wheel_friction prefix="front_right" dir="-1"/>
+  <xacro:wheel_friction prefix="rear_left" dir="-1"/>
+  <xacro:wheel_friction prefix="rear_right" dir="1"/>
   <ros2_control name="GazeboSimSystem" type="system">
     <hardware><plugin>gz_ros2_control/GazeboSimSystem</plugin></hardware>

Commit message: checkpoint: Ghost URDF must be built

File: src/velmobil_description/urdf/macros.urdf.xacro (robot description, xacro)
@@ -1,4 +1,4 @@
 <?xml version="1.0"?>
-<robot name="simple_velmobil" xmlns:xacro="http://www.ros.org/wiki/xacro" xmlns:gz="http://gazebosim.org/schema">
+<robot name="velmobil" xmlns:xacro="http://www.ros.org/wiki/xacro" xmlns:gz="http://gazebosim.org/schema">
     <xacro:macro name="wheel" params="prefix x y">
         <link name="${prefix}_wheel">

File: src/velmobil_description/urdf/properties.urdf.xacro (robot description, xacro)
@@ -1,4 +1,4 @@
 <?xml version="1.0"?>
-<robot name="simple_velmobil" xmlns:xacro="http://www.ros.org/wiki/xacro" xmlns:gz="http://gazebosim.org/schema">
+<robot name="velmobil" xmlns:xacro="http://www.ros.org/wiki/xacro" xmlns:gz="http://gazebosim.org/schema">
     <material name="orange"><color rgba="0.8 0.4 0.0 1.0"/></material>
     <material name="black"><color rgba="0 0 0 1.0"/></material>

File: src/velmobil_description/urdf/velmobil.urdf.xacro (robot description, xacro)
@@ -1,6 +1,7 @@
 <?xml version="1.0"?>
-<robot name="simple_velmobil" xmlns:xacro="http://www.ros.org/wiki/xacro" xmlns:gz="http://gazebosim.org/schema">
+<robot name="velmobil" xmlns:xacro="http://www.ros.org/wiki/xacro" xmlns:gz="http://gazebosim.org/schema">
   <xacro:include filename="$(find velmobil_description)/urdf/properties.urdf.xacro" />
   <xacro:include filename="$(find velmobil_description)/urdf/macros.urdf.xacro" />
+  <link name="world" />
   <link name="base_footprint" />
   <link name="base_link">
@@ -25,4 +26,9 @@
       <child link="base_link"/>
   </joint>
+  <joint name="world_base_joint" type="planar">
+    <origin xyz="0 0 0" rpy="0 0 0"/>
+    <parent link="world"/>
+    <child link="base_footprint"/>
+  </joint>
   <xacro:wheel prefix="front_left" x="0.5" y="${wheel_y_offset}"/>
   <xacro:wheel prefix="front_right" x="0.5" y="${-wheel_y_offset}"/>
@@ -42,5 +48,5 @@
   <gazebo>
     <plugin filename="gz_ros2_control-system" name="gz_ros2_control::GazeboSimROS2ControlPlugin">
-      <parameters>$(find velmobil_description)/control/simple_velmobil.yaml</parameters>
+      <parameters>$(find velmobil_description)/control_config/velmobil.yaml</parameters>
       <ros>
         <remapping>/mecanum_drive_controller/reference:=/cmd_vel</remapping>

Commit message: ghost velmobil (alpha)

File: src/velmobil_description/urdf/macros.urdf.xacro (robot description, xacro)
@@ -4,11 +4,11 @@
         <link name="${prefix}_wheel">
             <collision>
-                <origin xyz="0 0 0" rpy="${-pi/2} 0 0"/>
-                <geometry><cylinder length="0.1" radius="${wheel_radius}"/></geometry>
+                <origin xyz="0 0 0" rpy="0 0 0"/>
+                <geometry><sphere radius="${wheel_radius}"/></geometry>
             </collision>
             <visual>
-                <origin xyz="0 0 0" rpy="${-pi/2} 0 0"/>
+                <origin xyz="0 0 0" rpy="0 0 0"/>
                 <geometry>
-                    <cylinder length="0.1" radius="${wheel_radius}"/>
+                    <sphere radius="${wheel_radius}"/>
                 </geometry>
                 <material name="black"/>

File: src/velmobil_description/urdf/velmobil.urdf.xacro (robot description, xacro)
@@ -1,7 +1,7 @@
 <?xml version="1.0"?>
 <robot name="velmobil" xmlns:xacro="http://www.ros.org/wiki/xacro" xmlns:gz="http://gazebosim.org/schema">
+  <xacro:arg name="floating" default="true"/>
   <xacro:include filename="$(find velmobil_description)/urdf/properties.urdf.xacro" />
   <xacro:include filename="$(find velmobil_description)/urdf/macros.urdf.xacro" />
-  <link name="world" />
   <link name="base_footprint" />
   <link name="base_link">
@@ -26,9 +26,4 @@
       <child link="base_link"/>
   </joint>
-  <joint name="world_base_joint" type="planar">
-    <origin xyz="0 0 0" rpy="0 0 0"/>
-    <parent link="world"/>
-    <child link="base_footprint"/>
-  </joint>
   <xacro:wheel prefix="front_left" x="0.5" y="${wheel_y_offset}"/>
   <xacro:wheel prefix="front_right" x="0.5" y="${-wheel_y_offset}"/>
@@ -46,12 +41,21 @@
     <xacro:joint_interface name="rear_right_wheel_joint"/>
   </ros2_control>
-  <gazebo>
-    <plugin filename="gz_ros2_control-system" name="gz_ros2_control::GazeboSimROS2ControlPlugin">
-      <parameters>$(find velmobil_description)/control_config/velmobil.yaml</parameters>
-      <ros>
-        <remapping>/mecanum_drive_controller/reference:=/cmd_vel</remapping>
-        <remapping>/mecanum_drive_controller/odom:=/odom</remapping>
-      </ros>
-    </plugin>
-  </gazebo>
+  <xacro:if value="$(arg floating)">
+    <gazebo>
+      <plugin filename="gz_ros2_control-system" name="gz_ros2_control::GazeboSimROS2ControlPlugin">
+        <parameters>$(find velmobil_description)/control_config/floating_velmobil.yaml</parameters>
+      </plugin>
+    </gazebo>
+  </xacro:if>
+  <xacro:unless value="$(arg floating)">
+    <gazebo>
+      <plugin filename="gz_ros2_control-system" name="gz_ros2_control::GazeboSimROS2ControlPlugin">
+        <parameters>$(find velmobil_description)/control_config/velmobil.yaml</parameters>
+        <ros>
+          <remapping>/mecanum_drive_controller/reference:=/cmd_vel</remapping>
+          <remapping>/mecanum_drive_controller/odom:=/odom</remapping>
+        </ros>
+      </plugin>
+    </gazebo>
+  </xacro:unless>
 </robot>
