Commit message: full model pt.1

File: velmobil_description/urdf/macros.urdf.xacro (robot description, xacro)
@@ -20,5 +20,5 @@
         </link>
         <joint name="${prefix}_wheel_joint" type="continuous">
-            <origin xyz="${x} ${y} ${-wheel_base_offset}" rpy="0 0 0"/>
+            <origin xyz="${x} ${y} -0.02" rpy="0 0 0"/>
             <parent link="base_link"/>
             <child link="${prefix}_wheel"/>

File: velmobil_description/urdf/properties.urdf.xacro (robot description, xacro)
@@ -4,4 +4,11 @@
     <material name="black"><color rgba="0 0 0 1.0"/></material>
     <material name="white"><color rgba="1 1 1 1.0"/></material>
+    <xacro:property name="base_mass" value="60"/>
+    <xacro:property name="front_mass" value="15"/>
+    <xacro:property name="wheel_mass" value="1.6"/>
+    <xacro:property name="base_z_offset" value="0.1035"/>
+    <xacro:property name="base_link_center_offset" value="${base_z_offset - 0.019}"/>
+    <xacro:property name="base_center_offset" value="-0.081"/>
+    <xacro:property name="front_base_offset" value="0.445"/>
     <xacro:property name="wheel_radius" value="0.1016"/>
     <xacro:property name="lidar_l_centre_offset" value="0 0.3 0.176"/>
@@ -11,7 +18,7 @@
     <xacro:property name="imu_centre_ofset" value="0 0 0"/>
     <xacro:property name="wheel_y_offset" value="0.38"/>
-    <xacro:property name="wheel_centre_x_offset" value="0.36"/>
-    <xacro:property name="wheel_r_base_x_offset" value="${-wheel_centre_x_offset + 0.081}"/>
-    <xacro:property name="wheel_f_front_x_offset" value="${0.445 - 0.081 - wheel_centre_x_offset}"/>
+    <xacro:property name="wheel_center_x_offset" value="0.36"/>
+    <xacro:property name="wheel_r_base_x_offset" value="${-wheel_center_x_offset + 0.081}"/>
+    <xacro:property name="wheel_f_front_x_offset" value="${0.445 - 0.081 - wheel_center_x_offset}"/>
     <xacro:property name="wheel_base_offset" value="0.05"/>
 </robot>

File: velmobil_description/urdf/velmobil.urdf.xacro (robot description, xacro)
@@ -14,4 +14,5 @@
         <mesh filename="file://$(find velmobil_description)/models/base.dae" />
       </geometry>
+      <material name="orange"/>
     </visual>
     <inertial>
@@ -21,13 +22,35 @@
     </inertial>
   </link>
+  <link name="front_link">
+      <visual>
+          <geometry>
+              <mesh filename="file://$(find velmobil_description)/models/front.dae"/>
+          </geometry>
+          <material name="orange"/>
+      </visual>
+      <collision>
+          <geometry>
+              <mesh filename="file://$(find velmobil_description)/models/front.dae"/>
+          </geometry>
+      </collision>
+      <inertial>
+          <mass value="${front_mass}"/>
+          <inertia ixx="0.7351" ixy="0.0" ixz="0.0" iyy="0.0771" iyz="0.0" izz="0.7483"/>
+      </inertial>
+  </link>
   <joint name="footprint_joint" type="fixed">
-      <origin xyz="0 0 ${wheel_radius + wheel_base_offset}" rpy="0 0 0"/>
+      <origin xyz="${base_center_offset} 0 ${base_link_center_offset + 0.03}" rpy="0 0 0"/>
       <parent link="base_footprint"/>
       <child link="base_link"/>
   </joint>
-  <xacro:wheel prefix="front_left" x="0.5" y="${wheel_y_offset}"/>
-  <xacro:wheel prefix="front_right" x="0.5" y="${-wheel_y_offset}"/>
-  <xacro:wheel prefix="rear_left" x="-0.5" y="${wheel_y_offset}"/>
-  <xacro:wheel prefix="rear_right" x="-0.5" y="${-wheel_y_offset}"/>
+  <joint name="front_joint" type="fixed">
+      <origin xyz="${front_base_offset} 0 0" rpy="0 0 0"/>
+      <parent link="base_link"/>
+      <child link="front_link"/>
+  </joint>
+  <xacro:wheel prefix="front_left" x="${front_base_offset}" y="${wheel_y_offset}"/>
+  <xacro:wheel prefix="front_right" x="${front_base_offset}" y="${-wheel_y_offset}"/>
+  <xacro:wheel prefix="rear_left" x="${wheel_r_base_x_offset}" y="${wheel_y_offset}"/>
+  <xacro:wheel prefix="rear_right" x="${wheel_r_base_x_offset}" y="${-wheel_y_offset}"/>
   <xacro:wheel_friction prefix="front_left" dir="1"/>
   <xacro:wheel_friction prefix="front_right" dir="-1"/>

Commit message: lidar pt.2 + imu
Closes #11

File: velmobil_description/urdf/macros.urdf.xacro (robot description, xacro)
@@ -62,3 +62,130 @@
         </joint>
     </xacro:macro>
+    <xacro:macro name="lidar" params="name side yaw">
+        <link name="${name}_lidar_link">
+            <visual>
+                <geometry>
+                    <cylinder radius="${lidar_radius}" length="${lidar_length}"/>
+                </geometry>
+                <origin xyz="0 0 -0.02"/>
+                <material name="black"/>
+            </visual>
+            <collision>
+                <geometry>
+                    <cylinder radius="${lidar_radius}" length="${lidar_length}"/>
+                </geometry>
+            </collision>
+            <inertial>
+                <mass value="0.1"/>
+                <inertia ixx="0.00283314166" ixy="0.0" ixz="0.0" iyy="0.00283314166" iyz="0.0" izz="0.00143055"/>
+            </inertial>
+        </link>
+        <joint name="${name}_lidar_base_joint" type="fixed">
+            <parent link="base_link"/>
+            <child link="${name}_lidar_link"/>
+            <origin xyz="${-base_center_offset} ${side * lidar_y_offset} 0.176" rpy="0 0 ${yaw}"/>
+        </joint>
+        <gazebo reference="${name}_lidar_link">
+            <sensor name="${name}_lidar_sensor" type="gpu_lidar">
+                <ignition_frame_id>${name}_lidar_link</ignition_frame_id>
+                <pose relative_to='${name}_lidar_link'>0 0 0 0 0 0</pose>
+                <topic>/${name}/scan</topic>
+                <update_rate>50</update_rate>
+                <ray>
+                    <scan>
+                        <horizontal>
+                            <samples>540</samples>
+                            <resolution>1</resolution>
+                            <min_angle>-0.7853982</min_angle>
+                            <max_angle>3.926991</max_angle>
+                        </horizontal>
+                    </scan>
+                    <range>
+                        <min>0.06</min>
+                        <max>20</max>
+                        <resolution>0.01</resolution>
+                    </range>
+                    <noise>
+                        <type>gaussian</type>
+                        <mean>0.0</mean>
+                        <stddev>0.012</stddev>
+                    </noise>
+                </ray>
+                <always_on>1</always_on>
+                <visualize>1</visualize>
+            </sensor>
+        </gazebo>
+    </xacro:macro>
+    <xacro:macro name="imu" params="">
+        <link name="imu_link" />
+        <joint name="imu_base_link" type="fixed">
+            <parent link="base_link"/>
+            <child link="imu_link"/>
+            <origin xyz="0 0 0" rpy="0 0 0"/>
+        </joint>
+        <gazebo reference="imu_link">
+            <sensor name="imu_sensor" type="imu">
+                <ignition_frame_id>imu_link</ignition_frame_id>
+                <pose relative_to='imu_link'>0 0 0 0 0 0</pose>
+                <always_on>1</always_on>
+                <update_rate>1</update_rate>
+                <visualize>false</visualize>
+                <imu>
+                    <angular_velocity>
+                        <x>
+                            <noise type="gaussian">
+                                <mean>0.0</mean>
+                                <stddev>2e-4</stddev>
+                                <bias_mean>0.0000075</bias_mean>
+                                <bias_stddev>0.0000008</bias_stddev>
+                            </noise>
+                        </x>
+                        <y>
+                            <noise type="gaussian">
+                                <mean>0.0</mean>
+                                <stddev>2e-4</stddev>
+                                <bias_mean>0.0000075</bias_mean>
+                                <bias_stddev>0.0000008</bias_stddev>
+                            </noise>
+                        </y>
+                        <z>
+                            <noise type="gaussian">
+                                <mean>0.0</mean>
+                                <stddev>2e-4</stddev>
+                                <bias_mean>0.0000075</bias_mean>
+                                <bias_stddev>0.0000008</bias_stddev>
+                            </noise>
+                        </z>
+                    </angular_velocity>
+                    <linear_acceleration>
+                        <x>
+                            <noise type="gaussian">
+                                <mean>0.0</mean>
+                                <stddev>1.7e-2</stddev>
+                                <bias_mean>0.1</bias_mean>
+                                <bias_stddev>0.001</bias_stddev>
+                            </noise>
+                        </x>
+                        <y>
+                            <noise type="gaussian">
+                                <mean>0.0</mean>
+                                <stddev>1.7e-2</stddev>
+                                <bias_mean>0.1</bias_mean>
+                                <bias_stddev>0.001</bias_stddev>
+                            </noise>
+                        </y>
+                        <z>
+                            <noise type="gaussian">
+                                <mean>0.0</mean>
+                                <stddev>1.7e-2</stddev>
+                                <bias_mean>0.1</bias_mean>
+                                <bias_stddev>0.001</bias_stddev>
+                            </noise>
+                        </z>
+                    </linear_acceleration>
+                </imu>
+                <topic>/imu/data</topic>
+            </sensor>
+        </gazebo>
+    </xacro:macro>
 </robot>

File: velmobil_description/urdf/properties.urdf.xacro (robot description, xacro)
@@ -15,4 +15,5 @@
     <xacro:property name="lidar_l_orientation" value="0 0 0"/>
     <xacro:property name="lidar_r_centre_offset" value="0 -0.3 0.176"/>
+    <xacro:property name="lidar_y_offset" value="0.3"/>
     <xacro:property name="lidar_r_orientation" value="0 0 -3.141592"/>
     <xacro:property name="imu_centre_ofset" value="0 0 0"/>
@@ -22,3 +23,5 @@
     <xacro:property name="wheel_f_front_x_offset" value="${0.445 - 0.081 - wheel_center_x_offset}"/>
     <xacro:property name="wheel_base_offset" value="0.05"/>
+    <xacro:property name="lidar_radius" value="0.051"/>
+    <xacro:property name="lidar_length" value="0.152"/>
 </robot>

File: velmobil_description/urdf/velmobil.urdf.xacro (robot description, xacro)
@@ -57,4 +57,7 @@
   <xacro:wheel_friction prefix="rear_left" dir="-1"/>
   <xacro:wheel_friction prefix="rear_right" dir="1"/>
+  <xacro:lidar name="left" side="1" yaw="0.0" />
+  <xacro:lidar name="right" side="-1" yaw="-3.141592" />
+  <xacro:imu />
   <ros2_control name="GazeboSimSystem" type="system">
     <hardware><plugin>gz_ros2_control/GazeboSimSystem</plugin></hardware>

Commit message: firstly added realsense camera

File: velmobil_description/urdf/macros.urdf.xacro (robot description, xacro)
@@ -61,4 +61,71 @@
             <state_interface name="velocity"/>
         </joint>
+    </xacro:macro>
+    <xacro:macro name="real_sense" params="">
+        <joint name="rgbd_camera_joint" type="fixed">
+            <origin xyz="0.45 0 0.09" rpy="0 0 0"/>
+            <parent link="base_link"/>
+            <child link="rgbd_camera_frame"/>
+        </joint>
+        <link name="rgbd_camera_frame">
+        <visual>
+            <origin xyz="0 0 0" rpy="0 0 0"/>
+            <geometry>
+            <mesh filename="file://$(find velmobil_description)/models/real_sense.dae" scale="1.0 1.0 1.0"/>
+            </geometry>
+            <material name="black">
+            <color rgba="0.9 0.9 0.9 1.0"/>
+            </material>
+        </visual>
+        </link>
+        <gazebo reference="rgbd_camera_frame">
+        <sensor name="rgbd_camera" type="rgbd_camera">
+            <ignition_frame_id>rgbd_camera_frame</ignition_frame_id>
+            <camera name="rgbd_camera_frame">
+            <horizontal_fov>1.3962634</horizontal_fov>
+            <lens>
+                <intrinsics>
+                <fx>277.1</fx>
+                <fy>277.1</fy>
+                <cx>160.5</cx>
+                <cy>120.5</cy>
+                <s>0</s>
+                </intrinsics>
+            </lens>
+            <distortion>
+                <k1>0.104207</k1>
+                <k2>-0.255558</k2>
+                <k3>0.128694</k3>
+                <p1>0.000512</p1>
+                <p2>0.000319</p2>
+                <center>0.5 0.5</center>
+            </distortion>
+            <image>
+                <width>1280</width>
+                <height>720</height>
+                <format>L8</format>
+            </image>
+            <clip>
+                <near>0.01</near>
+                <far>300</far>
+            </clip>
+            <depth_camera>
+                <clip>
+                <near>0.1</near>
+                <far>10</far>
+                </clip>
+            </depth_camera>
+            <noise>
+                <type>gaussian</type>
+                <mean>0</mean>
+                <stddev>0.003</stddev>
+            </noise>
+            </camera>
+            <always_on>1</always_on>
+            <update_rate>10</update_rate>
+            <visualize>0</visualize>
+            <topic>depth_camera</topic>
+        </sensor>
+        </gazebo>
     </xacro:macro>
     <xacro:macro name="lidar" params="name side yaw">

File: velmobil_description/urdf/velmobil.urdf.xacro (robot description, xacro)
@@ -60,4 +60,5 @@
   <xacro:lidar name="right" side="-1" yaw="-3.141592" />
   <xacro:imu />
+  <xacro:real_sense />
   <ros2_control name="GazeboSimSystem" type="system">
     <hardware><plugin>gz_ros2_control/GazeboSimSystem</plugin></hardware>

Commit message: added second camera and camera base in order to fix camera to them - almost like in real velmobil

File: velmobil_description/urdf/macros.urdf.xacro (robot description, xacro)
@@ -25,4 +25,11 @@
             <axis xyz="0 1 0"/>
             <dynamics damping="0.2"/>
+        </joint>
+    </xacro:macro>
+    <xacro:macro name="camera_link_camera_joint" params="prefix">
+        <joint name="${prefix}_camera_link_camera_joint" type="fixed">
+            <origin xyz="0 0 0" rpy="0 0 0"/>
+            <parent link="camera_link"/>
+            <child link="${prefix}_rgbd_camera_frame"/>
         </joint>
     </xacro:macro>
@@ -62,11 +69,12 @@
         </joint>
     </xacro:macro>
-    <xacro:macro name="real_sense" params="">
-        <joint name="rgbd_camera_joint" type="fixed">
-            <origin xyz="0.45 0 0.09" rpy="0 0 0"/>
-            <parent link="base_link"/>
-            <child link="rgbd_camera_frame"/>
-        </joint>
-        <link name="rgbd_camera_frame">
+    <!-- TWO CAMERAS SHOULD ARE SET FOR EVEN OPTIMAL WORKING WHILE SIMULATION -->
+    <xacro:macro name="front_real_sense" params="">
+        <joint name="front_rgbd_camera_joint" type="fixed">
+            <origin xyz="${-base_center_offset + 0.2} 0 0.14" rpy="0 0 0"/>
+            <parent link="camera_link"/>
+            <child link="front_rgbd_camera_frame"/>
+        </joint>
+        <link name="front_rgbd_camera_frame">
         <visual>
             <origin xyz="0 0 0" rpy="0 0 0"/>
@@ -79,51 +87,62 @@
         </visual>
         </link>
-        <gazebo reference="rgbd_camera_frame">
-        <sensor name="rgbd_camera" type="rgbd_camera">
-            <ignition_frame_id>rgbd_camera_frame</ignition_frame_id>
-            <camera name="rgbd_camera_frame">
-            <horizontal_fov>1.3962634</horizontal_fov>
-            <lens>
-                <intrinsics>
-                <fx>277.1</fx>
-                <fy>277.1</fy>
-                <cx>160.5</cx>
-                <cy>120.5</cy>
-                <s>0</s>
-                </intrinsics>
-            </lens>
-            <distortion>
-                <k1>0.104207</k1>
-                <k2>-0.255558</k2>
-                <k3>0.128694</k3>
-                <p1>0.000512</p1>
-                <p2>0.000319</p2>
-                <center>0.5 0.5</center>
-            </distortion>
+        <gazebo reference="front_rgbd_camera_frame">
+        <sensor name="front_rgbd_camera" type="rgbd_camera">
+            <ignition_frame_id>front_rgbd_camera_frame</ignition_frame_id>
+            <camera name="front_rgbd_camera_frame">
+            <horizontal_fov>1.094321441</horizontal_fov>
             <image>
-                <width>1280</width>
-                <height>720</height>
-                <format>L8</format>
+                <width>320</width>
+                <height>180</height>
+                <format>R8G8B8</format>
             </image>
             <clip>
-                <near>0.01</near>
-                <far>300</far>
+                <near>0.4</near>
+                <far>6.5</far>
             </clip>
-            <depth_camera>
-                <clip>
-                <near>0.1</near>
-                <far>10</far>
-                </clip>
-            </depth_camera>
-            <noise>
-                <type>gaussian</type>
-                <mean>0</mean>
-                <stddev>0.003</stddev>
-            </noise>
             </camera>
             <always_on>1</always_on>
             <update_rate>10</update_rate>
             <visualize>0</visualize>
-            <topic>depth_camera</topic>
+            <topic>front_depth_camera</topic>
+        </sensor>
+        </gazebo>
+    </xacro:macro>
+    <xacro:macro name="back_real_sense" params="">
+        <joint name="back_rgbd_camera_joint" type="fixed">
+            <origin xyz="${-base_center_offset - 0.2} 0 0.14" rpy="0 0 -3.14"/>
+            <parent link="camera_link"/>
+            <child link="back_rgbd_camera_frame"/>
+        </joint>
+        <link name="back_rgbd_camera_frame">
+        <visual>
+            <origin xyz="0 0 0" rpy="0 0 0"/>
+            <geometry>
+            <mesh filename="file://$(find velmobil_description)/models/real_sense.dae" scale="1.0 1.0 1.0"/>
+            </geometry>
+            <material name="black">
+            <color rgba="0.9 0.9 0.9 1.0"/>
+            </material>
+        </visual>
+        </link>
+        <gazebo reference="back_rgbd_camera_frame">
+        <sensor name="back_rgbd_camera" type="rgbd_camera">
+            <ignition_frame_id>back_rgbd_camera_frame</ignition_frame_id>
+            <camera name="back_rgbd_camera_frame">
+            <horizontal_fov>1.094321441</horizontal_fov>
+            <image>
+                <width>320</width>
+                <height>180</height>
+                <format>R8G8B8</format>
+            </image>
+            <clip>
+                <near>0.4</near>
+                <far>6.5</far>
+            </clip>
+            </camera>
+            <always_on>1</always_on>
+            <update_rate>10</update_rate>
+            <visualize>0</visualize>
+            <topic>back_depth_camera</topic>
         </sensor>
         </gazebo>

File: velmobil_description/urdf/properties.urdf.xacro (robot description, xacro)
@@ -7,4 +7,7 @@
     <xacro:property name="front_mass" value="15"/>
     <xacro:property name="wheel_mass" value="1.6"/>
+    <xacro:property name="base_link_width" value="0.7604" />
+    <xacro:property name="base_link_height" value="0.7203" />
+    <xacro:property name="base_link_depth" value="0.1598" />
     <xacro:property name="base_z_offset" value="0.1035"/>
     <xacro:property name="base_link_center_offset" value="${base_z_offset - 0.019}"/>

File: velmobil_description/urdf/velmobil.urdf.xacro (robot description, xacro)
@@ -6,8 +6,4 @@
   <link name="base_footprint" />
   <link name="base_link">
-    <collision>
-      <origin xyz="0 0 0.5" rpy="0 0 0"/>
-      <geometry><box size="0.1 0.1 0.1"/></geometry>  <!-- mock colision -->
-    </collision>
     <visual>
       <geometry>
@@ -16,4 +12,10 @@
       <material name="orange"/>
     </visual>
+    <collision>
+      <origin xyz="0 -0.011 0.001" rpy="0 0 0"/>
+      <geometry>
+        <box size="${base_link_width} ${base_link_height} ${base_link_depth}"/>
+      </geometry>
+    </collision>
     <inertial>
       <origin xyz="0 0 0.5" rpy="0 0 0"/>
@@ -30,6 +32,7 @@
       </visual>
       <collision>
+          <origin xyz="0.0 0.003 0.002" rpy="0.0 0.0 1.57"/>
           <geometry>
-              <mesh filename="file://$(find velmobil_description)/models/front.dae"/>
+              <box size="0.6736 0.1906 0.1600"/>
           </geometry>
       </collision>
@@ -60,5 +63,31 @@
   <xacro:lidar name="right" side="-1" yaw="-3.141592" />
   <xacro:imu />
-  <xacro:real_sense />
+  <link name="camera_link">
+    <collision>
+        <origin xyz="${-base_center_offset} 0 0" rpy="0 0 1.57"/>
+        <geometry>
+            <box size="0.1 0.2 0.2"/>
+        </geometry>
+    </collision>
+    <visual>
+        <origin xyz="${-base_center_offset} 0 0" rpy="0 0 1.57"/>
+        <geometry>
+            <box size="0.2 0.38 0.3"/>
+        </geometry>
+        <material name="orange"/>
+    </visual>
+    <inertial>
+        <mass value="5.0"/>
+        <inertia ixx="0.1" ixy="0.0" ixz="0.0"
+                 iyy="0.1" iyz="0.0" izz="0.1"/>
+    </inertial>
+  </link>
+  <joint name="base_camera_link" type="fixed">
+      <origin xyz="0 0 0.15" rpy="0 0 0"/>
+      <parent link="base_link"/>
+      <child link="camera_link"/>
+  </joint>
+  <xacro:front_real_sense />
+  <xacro:back_real_sense />
   <ros2_control name="GazeboSimSystem" type="system">
     <hardware><plugin>gz_ros2_control/GazeboSimSystem</plugin></hardware>
