Commit message: changed camera link orientation on velmobil

File: velmobil_description/urdf/macros.urdf.xacro (robot description, xacro)
@@ -72,5 +72,5 @@
     <xacro:macro name="front_real_sense" params="">
         <joint name="front_rgbd_camera_joint" type="fixed">
-            <origin xyz="${-base_center_offset + 0.2} 0 0.14" rpy="0 0 0"/>
+            <origin xyz="${-base_center_offset + 0.1} 0 0.14" rpy="0 0 0"/>
             <parent link="camera_link"/>
             <child link="front_rgbd_camera_frame"/>
@@ -111,5 +111,5 @@
     <xacro:macro name="back_real_sense" params="">
         <joint name="back_rgbd_camera_joint" type="fixed">
-            <origin xyz="${-base_center_offset - 0.2} 0 0.14" rpy="0 0 -3.14"/>
+            <origin xyz="${-base_center_offset - 0.1} 0 0.14" rpy="0 0 -3.14"/>
             <parent link="camera_link"/>
             <child link="back_rgbd_camera_frame"/>

File: velmobil_description/urdf/velmobil.urdf.xacro (robot description, xacro)
@@ -65,5 +65,5 @@
   <link name="camera_link">
     <collision>
-        <origin xyz="${-base_center_offset} 0 0" rpy="0 0 1.57"/>
+        <origin xyz="${-base_center_offset} 0 0" rpy="0 0 0"/>
         <geometry>
             <box size="0.1 0.2 0.2"/>
@@ -71,5 +71,5 @@
     </collision>
     <visual>
-        <origin xyz="${-base_center_offset} 0 0" rpy="0 0 1.57"/>
+        <origin xyz="${-base_center_offset} 0 0" rpy="0 0 0"/>
         <geometry>
             <box size="0.2 0.38 0.3"/>
