Commit message: feat(urdf): added yaw joints to model #42

File: velmobil_description/urdf/macros.urdf.xacro (robot description, xacro)
@@ -2,4 +2,12 @@
 <robot name="velmobil" xmlns:xacro="http://www.ros.org/wiki/xacro" xmlns:gz="http://gazebosim.org/schema">
     <xacro:macro name="wheel" params="prefix x y">
+        <link name="${prefix}_yaw">
+            <!-- useless, but urdf->sdf won't happen without mock inertia -->
+            <inertial>
+                <mass value="0.0001"/>
+                <origin xyz="0 0 0" rpy="0 0 0"/>
+                <inertia ixx="0.000001" ixy="0.0" ixz="0.0" iyy="0.000001" iyz="0.0" izz="0.000001"/>
+            </inertial>
+        </link>
         <link name="${prefix}_wheel">
             <collision>
@@ -19,7 +27,14 @@
             </inertial>
         </link>
-        <joint name="${prefix}_wheel_joint" type="continuous">
+        <joint name="${prefix}_yaw_joint" type="revolute">
             <origin xyz="${x} ${y} -0.02" rpy="0 0 0"/>
             <parent link="base_link"/>
+            <child link="${prefix}_yaw"/>
+            <axis xyz="0 0 1"/>
+            <limit lower="${-pi}" upper="${pi}" effort="100000" velocity="10000"/>
+        </joint>
+        <joint name="${prefix}_wheel_joint" type="continuous">
+            <origin xyz="0 0 0" rpy="0 0 0"/>
+            <parent link="${prefix}_yaw"/>
             <child link="${prefix}_wheel"/>
             <axis xyz="0 1 0"/>
@@ -59,5 +74,5 @@
         </gazebo>
     </xacro:macro>
-    <xacro:macro name="joint_interface" params="name">
+    <xacro:macro name="wheel_joint_interface" params="name">
         <joint name="${name}">
             <command_interface name="velocity">
@@ -67,4 +82,13 @@
             <state_interface name="position"/>
             <state_interface name="velocity"/>
+        </joint>
+    </xacro:macro>
+    <xacro:macro name="yaw_joint_interface" params="name">
+        <joint name="${name}">
+            <command_interface name="position">
+                <param name="min">${-pi}</param>
+                <param name="max">${pi}</param>
+            </command_interface>
+            <state_interface name="position"/>
         </joint>
     </xacro:macro>

File: velmobil_description/urdf/velmobil.urdf.xacro (robot description, xacro)
@@ -92,8 +92,12 @@
   <ros2_control name="GazeboSimSystem" type="system">
     <hardware><plugin>gz_ros2_control/GazeboSimSystem</plugin></hardware>
-    <xacro:joint_interface name="front_left_wheel_joint"/>
-    <xacro:joint_interface name="front_right_wheel_joint"/>
-    <xacro:joint_interface name="rear_left_wheel_joint"/>
-    <xacro:joint_interface name="rear_right_wheel_joint"/>
+    <xacro:wheel_joint_interface name="front_left_wheel_joint"/>
+    <xacro:wheel_joint_interface name="front_right_wheel_joint"/>
+    <xacro:wheel_joint_interface name="rear_left_wheel_joint"/>
+    <xacro:wheel_joint_interface name="rear_right_wheel_joint"/>
+    <xacro:yaw_joint_interface name="front_left_yaw_joint"/>
+    <xacro:yaw_joint_interface name="front_right_yaw_joint"/>
+    <xacro:yaw_joint_interface name="rear_left_yaw_joint"/>
+    <xacro:yaw_joint_interface name="rear_right_yaw_joint"/>
   </ros2_control>
   <xacro:if value="$(arg floating)">
@@ -128,4 +132,8 @@
         <joint_name>rear_left_wheel_joint</joint_name>
         <joint_name>rear_right_wheel_joint</joint_name>
+        <joint_name>front_left_yaw_joint</joint_name>
+        <joint_name>front_right_yaw_joint</joint_name>
+        <joint_name>rear_left_yaw_joint</joint_name>
+        <joint_name>rear_right_yaw_joint</joint_name>
       </plugin>
     </gazebo>

Commit message: feat(ros2_control): Improved roll_yaw_controller, repaired y-slip-bug #19

File: velmobil_description/urdf/macros.urdf.xacro (robot description, xacro)
@@ -49,5 +49,5 @@
         </joint>
     </xacro:macro>
-    <xacro:macro name="wheel_friction" params="prefix dir">
+    <xacro:macro name="wheel_friction" params="prefix">
         <gazebo reference="${prefix}_wheel">
             <collision>
@@ -56,8 +56,8 @@
                         <ode>
                             <mu>1.0</mu>
-                            <mu2>0.01</mu2>
-                            <fdir1 gz:expressed_in="base_link">1 ${dir} 0</fdir1>
+                            <mu2>1.0</mu2>
+                            <fdir1 gz:expressed_in="${prefix}_yaw">1 0 0</fdir1>
                             <slip1>0.0</slip1>
-                            <slip2>0.5</slip2>
+                            <slip2>0.0</slip2>
                         </ode>
                     </friction>

File: velmobil_description/urdf/velmobil.urdf.xacro (robot description, xacro)
@@ -58,8 +58,8 @@
   <xacro:wheel prefix="rear_left" x="${wheel_r_base_x_offset}" y="${wheel_y_offset}"/>
   <xacro:wheel prefix="rear_right" x="${wheel_r_base_x_offset}" y="${-wheel_y_offset}"/>
-  <xacro:wheel_friction prefix="front_left" dir="-1"/>
-  <xacro:wheel_friction prefix="front_right" dir="1"/>
-  <xacro:wheel_friction prefix="rear_left" dir="1"/>
-  <xacro:wheel_friction prefix="rear_right" dir="-1"/>
+  <xacro:wheel_friction prefix="front_left"/>
+  <xacro:wheel_friction prefix="front_right"/>
+  <xacro:wheel_friction prefix="rear_left"/>
+  <xacro:wheel_friction prefix="rear_right"/>
   <xacro:lidar name="left" side="1" yaw="0.0" />
   <xacro:lidar name="right" side="-1" yaw="-3.141592" />

Commit message: added macro to get velmobil ground truth position

File: velmobil_description/urdf/macros.urdf.xacro (robot description, xacro)
@@ -299,3 +299,15 @@
         </gazebo>
     </xacro:macro>
+    <xacro:macro name="ground_truth" params="topic:=/gt_position freq:=50">
+        <gazebo>
+            <plugin filename="gz-sim-odometry-publisher-system"
+                    name="gz::sim::systems::OdometryPublisher">
+            <odom_frame>odom</odom_frame>
+            <robot_base_frame>base_link</robot_base_frame>
+            <odom_topic>${topic}</odom_topic>
+            <odom_publish_frequency>${freq}</odom_publish_frequency>
+            <dimensions>3</dimensions>
+            </plugin>
+        </gazebo>
+    </xacro:macro>
 </robot>

File: velmobil_description/urdf/velmobil.urdf.xacro (robot description, xacro)
@@ -65,4 +65,5 @@
   <xacro:lidar name="right" side="-1" yaw="-3.141592" />
   <xacro:imu />
+  <xacro:ground_truth/>
   <link name="camera_link">
     <collision>

Commit message: dev(agent + model): Added SBX library and repaired velmobil chassis mass

File: velmobil_description/urdf/macros.urdf.xacro (robot description, xacro)
@@ -23,5 +23,5 @@
             </visual>
             <inertial>
-                <mass value="1.0"/>
+                <mass value="${wheel_mass}"/>
                 <inertia ixx="0.145" ixy="0.0" ixz="0.0" iyy="0.145" iyz="0.0" izz="0.125"/>
             </inertial>

File: velmobil_description/urdf/velmobil.urdf.xacro (robot description, xacro)
@@ -22,5 +22,5 @@
     <inertial>
       <origin xyz="0 0 0.5" rpy="0 0 0"/>
-      <mass value="0.5"/>
+      <mass value="${base_mass}"/>
       <inertia ixx="0.13" ixy="0.0" ixz="0.0" iyy="0.42" iyz="0.0" izz="0.48"/>
     </inertial>
