Commit message: dev(agent+sim_man): Agent learns

File: velmobil_description/urdf/properties.urdf.xacro (robot description, xacro)
@@ -4,7 +4,7 @@
     <material name="black"><color rgba="0 0 0 1.0"/></material>
     <material name="white"><color rgba="1 1 1 1.0"/></material>
-    <xacro:property name="base_mass" value="60"/>
-    <xacro:property name="front_mass" value="15"/>
-    <xacro:property name="wheel_mass" value="1.6"/>
+    <xacro:property name="base_mass" value="100"/>
+    <xacro:property name="front_mass" value="30"/>
+    <xacro:property name="wheel_mass" value="0.1"/>
     <xacro:property name="base_link_width" value="0.7604" />
     <xacro:property name="base_link_height" value="0.7203" />
